Commit message: added back asus sensor

File: r2_gazebo/robots/r2.sim.urdf.xacro (robot description, xacro)
@@ -7,6 +7,5 @@
   <xacro:include filename="$(find r2_description)/robots/r2.urdf.xacro" />
    <xacro:include filename="$(find r2_gazebo)/urdf/r2.gazebo.xacro" />
-<!--   <xacro:include filename="$(find r2_gazebo)/urdf/sensors/r2.gazebo.sensors.xacro" />
- -->
+  <xacro:include filename="$(find r2_gazebo)/urdf/sensors/r2.gazebo.sensors.xacro" />
   <xacro:include filename="$(find r2_gazebo)/urdf/gazebo_plugins/r2.transmissions.xacro" />
   <xacro:include filename="$(find r2_gazebo)/urdf/gazebo_plugins/r2.gazebo.controller.xacro" />

File: r2_gazebo/urdf/sensors/asus.gazebo.xacro (robot description, xacro)
@@ -1,3 +1,133 @@
-<?xml version="1.0"?>
+<?xml version="1.0" ?>
+<robot xmlns:xacro="http://www.ros.org/wiki/xacro" name="r2">
+  <!--
+  ASUS Xtion PRO LIVE
+    Specs from:
+    http://www.asus.com/Multimedia/Xtion_PRO_LIVE/#specifications
+  -->
+  <xacro:property name="AsusWidth" value="0.018"/>
+  <xacro:property name="AsusHeight" value="0.035"/>
+  <xacro:property name="AsusDepth" value="0.05"/>
+  <xacro:property name="AsusMass" value="0.25"/>
+  <xacro:property name="AsusImageWidth" value="640"/>
+  <xacro:property name="AsusImageHeight" value="480"/>
+  <xacro:property name="AsusFieldOfView" value="1.01229097"/>
+  <xacro:property name="AsusMinDistance" value="0.2"/>
+  <xacro:property name="AsusMaxDistance" value="5"/>
+  <xacro:property name="AsusFrameRate" value="30"/>
+  <xacro:macro name="asus_sensor" params="sensor_name parent_camera_link parent_depth_link">
+    <!-- <xacro:virtual_link name="${sensor_name}_Frame"
+                    origin_rpy="0 0 0"
+                    origin_xyz="0 0 0"/>
+ -->
+      <gazebo reference="${parent_camera_link}">
+        <sensor type="depth" name="openni_camera_camera">
+            <always_on>1</always_on>
+            <visualize>true</visualize>
+            <camera>
+                <horizontal_fov>1.047</horizontal_fov>
+                <image>
+                    <width>1280</width>
+                    <height>960</height>
+                    <format>R8G8B8</format>
+                </image>
+                <depth_camera> </depth_camera>
+                <clip>
+                    <near>0.1</near>
+                    <far>100</far>
+                </clip>
+            </camera>
+            <plugin name="camera_controller" filename="libgazebo_ros_openni_kinect.so">
+                <alwaysOn>true</alwaysOn>
+                <updateRate>2.0</updateRate>
+                <cameraName>${sensor_name}</cameraName>
+                <frameName>${parent_depth_link}</frameName>
+                <imageTopicName>/${sensor_name}/rgb/image_raw</imageTopicName>
+                <depthImageTopicName>/${sensor_name}/depth/image_raw</depthImageTopicName>
+                <pointCloudTopicName>/${sensor_name}/depth/points</pointCloudTopicName>
+                <cameraInfoTopicName>/${sensor_name}/rgb/camera_info</cameraInfoTopicName>
+                <depthImageCameraInfoTopicName>/${sensor_name}/depth/camera_info</depthImageCameraInfoTopicName>
+                <pointCloudCutoff>0.4</pointCloudCutoff>
+                <hackBaseline>0.0</hackBaseline>
+                <distortionK1>0.0</distortionK1>
+                <distortionK2>0.0</distortionK2>
+                <distortionK3>0.0</distortionK3>
+                <distortionT1>0.0</distortionT1>
+                <distortionT2>0.0</distortionT2>
+                <CxPrime>0.0</CxPrime>
+                <Cx>0.0</Cx>
+                <Cy>0.0</Cy>
+                <focalLength>0.0</focalLength>
+                </plugin>
+        </sensor>
+    </gazebo>
+<!--
+      <gazebo>
+      <plugin name="head_camera_controller" filename="libgazebo_ros_openni_kinect.so">
+        <baseline>0.2</baseline>
+        <alwaysOn>true</alwaysOn>
+        <updateRate>1.0</updateRate>
+        <cameraName>${sensor_name}</cameraName>
+        <imageTopicName>/${sensor_name}/depth/image_raw</imageTopicName>
+        <cameraInfoTopicName>/${sensor_name}/depth/camera_info</cameraInfoTopicName>
+        <depthImageTopicName>/${sensor_name}/depth/image_raw</depthImageTopicName>
+        <depthImageInfoTopicName>/${sensor_name}/depth/camera_info</depthImageInfoTopicName>
+        <pointCloudTopicName>/${sensor_name}/depth/points</pointCloudTopicName>
+        <frameName>/${parent_link}/${sensor_name}</frameName>
+        <pointCloudCutoff>0.5</pointCloudCutoff>
+        <distortionK1>0.00000001</distortionK1>
+        <distortionK2>0.00000001</distortionK2>
+        <distortionK3>0.00000001</distortionK3>
+        <distortionT1>0.00000001</distortionT1>
+        <distortionT2>0.00000001</distortionT2>
+        <CxPrime>0</CxPrime>
+        <Cx>0</Cx>
+        <Cy>0</Cy>
+        <focalLength>0</focalLength>
+        <hackBaseline>0</hackBaseline>
+      </plugin> -->
+    <!-- <gazebo reference="${sensor_name}_Frame">
+      <sensor name="asus/ir" type="depth">
+        <camera>
+          <image>
+            <width>${AsusImageWidth}</width>
+            <height>${AsusImageHeight}</height>
+            <format>R8G8B8</format>
+          </image>
+          <horizontal_fov>${AsusFieldOfView}</horizontal_fov>
+          <clip>
+            <near>${AsusMinDistance}</near>
+            <far>${AsusMaxDistance}</far>
+          </clip>
+        </camera>
+        <update_rate>${AsusFrameRate}</update_rate>
+        <plugin filename="libAsusXtionPluginRos.so" name="${sensor_name}_Controller">
+          <updateRate>${AsusFrameRate}</updateRate>
+          <cameraName>${sensor_name}</cameraName>
+          <imageTopicName>rgb/image_raw</imageTopicName>
+          <cameraInfoTopicName>rgb/camera_info</cameraInfoTopicName>
+          <depthImageTopicName>depth/image_raw</depthImageTopicName>
+          <depthCameraInfoTopicName>depth/camera_info</depthCameraInfoTopicName>
+          <pointCloudTopicName>depth/points</pointCloudTopicName>
+          <frameName>${sensor_name}IR_Frame</frameName>
+          <pointCloudCutoff>0.2</pointCloudCutoff>
+          <hack_baseline>0.2</hack_baseline>
+        </plugin>
+      </sensor>
+    </gazebo> -->
+    <!-- <xacro:fixed_joint jointName="${sensor_name}_Offset"
+                       parent="${parent_link}" child="${sensor_name}_Frame"
+                       origin_rpy="${origin_rpy}"
+                       origin_xyz="${origin_xyz}"/>
+    <xacro:virtual_link name="${sensor_name}IR_Frame"
+                    origin_rpy="0 0 0"
+                    origin_xyz="0 0 0"/>
+    <xacro:fixed_joint jointName="${sensor_name}IR_Offset"
+                       parent="${sensor_name}_Frame" child="${sensor_name}IR_Frame"
+                       origin_rpy="-1.57 0 -1.57"
+                       origin_xyz="0 0 0"/> -->
+  </xacro:macro>
+</robot>
+<!-- <?xml version="1.0"?>
 <root xmlns:sensor="http://playerstage.sourceforge.net/gazebo/xmlschema/#sensor"
       xmlns:controller="http://playerstage.sourceforge.net/gazebo/xmlschema/#controller"
@@ -65,2 +195,3 @@
     </xacro:macro>
 </root>
+ -->

File: r2_gazebo/urdf/sensors/r2.gazebo.sensors.xacro (robot description, xacro)
@@ -4,60 +4,10 @@
 			xmlns:sensor="http://playerstage.sourceforge.net/gazebo/xmlschema/#sensor"
 			xmlns:xacro="http://playerstage.sourceforge.net/gazebo/xmlschema/#interface">
-  <xacro:include filename="$(find r2_gazebo)/urdf/sensors/grasshopper2.gazebo.xacro" />
-  <xacro:include filename="$(find r2_gazebo)/urdf/sensors/asus.gazebo.xacro" />
-  <xacro:grasshopper2_cam_gazebo_v0 camera_name="${robot_name}neck/head/camera0" frame_name="${robot_name}left_camera_optical_frame" />
+<!--   <xacro:include filename="$(find r2_gazebo)/urdf/sensors/grasshopper2.gazebo.xacro" />
+ -->
+ <xacro:include filename="$(find r2_gazebo)/urdf/sensors/asus.gazebo.xacro" />
+<!--   <xacro:grasshopper2_cam_gazebo_v0 camera_name="${robot_name}neck/head/camera0" frame_name="${robot_name}left_camera_optical_frame" />
   <xacro:grasshopper2_cam_gazebo_v0 camera_name="${robot_name}neck/head/camera1" frame_name="${robot_name}right_camera_optical_frame" />
-  <xacro:macro name="asus_camera" params="name parent cam_name">
-    <joint name="${name}_ir_joint" type="fixed">
-      <!-- <origin xyz="-0.032267 0.0125 0.136453" rpy="0 0 0"/> -->
-      <origin xyz="0 0 0" rpy="0 0 0"/>
-      <parent link="${parent}"/>
-      <child link="${name}_ir_link"/>
-    </joint>
-    <link name="${name}_ir_link">
-      <inertial>
-        <mass value="0.1" />
-        <origin xyz="0 0 0" rpy="0 0 0"/>
-        <inertia ixx="0.01"  ixy="0.0"  ixz="0.0"
-                 iyy="0.01"  iyz="0.0"
-                 izz="0.01" />
-      </inertial>
-    </link>
-    <joint name="${name}_ir_optical_frame_joint" type="fixed">
-      <origin xyz="0 0 0" rpy="-1.57 0 -1.57" /> <!-- this works for non-rgb 3d data... -->
-      <parent link="${name}_ir_link"/>
-      <child link="${name}_ir_optical_frame"/>
-    </joint>
-    <link name="${name}_ir_optical_frame">
-      <inertial>
-        <mass value=".1"/>
-        <inertia ixx=".0010" ixy="0.0" ixz="0.0" iyy=".0010" iyz="0.0" izz=".0010"/>
-      </inertial>
-    </link>
-    <xacro:asus_ir_gazebo_v0 link_name="${name}_ir_link" frame_name="${name}_ir_optical_frame" camera_name="${cam_name}" />
-    <joint name="${name}_rgb_joint" type="fixed">
-      <origin xyz="0 -0.03 0" rpy="3.14 0 0"/>
-      <parent link="${name}_ir_link"/>
-      <child link="${name}_rgb_link"/>
-    </joint>
-    <link name="${name}_rgb_link" >
-      <inertial>
-      <mass value=".1"/>
-      <inertia ixx=".0010" ixy="0.0" ixz="0.0" iyy=".0010" iyz="0.0" izz=".0010"/>
-      </inertial>
-    </link>
-    <joint name="${name}_rgb_optical_frame_joint" type="fixed">
-       <origin xyz="0 0 0" rpy="-1.57 0 -1.57" />
-      <parent link="${name}_rgb_link"/>
-      <child link="${name}_rgb_optical_frame"/>
-    </joint>
-    <link name="${name}_rgb_optical_frame">
-        <inertial>
-          <mass value=".1"/>
-          <inertia ixx=".0010" ixy="0.0" ixz="0.0" iyy=".0010" iyz="0.0" izz=".0010"/>
-        </inertial>
-    </link>
-    <xacro:asus_rgb_gazebo_v0 link_name="${name}_rgb_link" frame_name="${name}_rgb_optical_frame" camera_name="${cam_name}" />
-  </xacro:macro>
-  <xacro:asus_camera name="asus" parent="${robot_name}simulated_asus_frame" cam_name="${robot_name}neck/head/range_camera0"/>
+ -->
+  <xacro:asus_sensor sensor_name="${robot_name}asus" parent_camera_link="${robot_name}simulated_asus_camera_frame" parent_depth_link="${robot_name}simulated_asus_depth_frame"/>
 </robot>
