Commit message: added leg sensors for hydro. changed lasers to "camboard nanos" (i.e., short range PC devices). also removed one of the two cameras on feet.

File: r2_gazebo/robots/r2_fullbody.sim.urdf.xacro (robot description, xacro)
@@ -7,10 +7,9 @@
   <xacro:include filename="$(find r2_description)/robots/r2_fullbody.urdf.xacro" />
   <xacro:include filename="$(find r2_gazebo)/urdf/r2.gazebo.xacro" />
-<!--   <xacro:include filename="$(find r2_gazebo)/urdf/sensors/r2.gazebo.sensors.xacro" />
- -->
+  <xacro:include filename="$(find r2_gazebo)/urdf/sensors/r2.gazebo.sensors.xacro" />
   <xacro:include filename="$(find r2_gazebo)/urdf/r2_legs.gazebo.xacro" />
-<!--   <xacro:include filename="$(find r2_gazebo)/urdf/sensors/r2_legs.gazebo.sensors.xacro" />
- -->
-  <!-- <xacro:include filename="$(find r2_gazebo)/urdf/gazebo_plugins/p3d_base_controller.xacro" />
+  <xacro:include filename="$(find r2_gazebo)/urdf/sensors/r2_legs.gazebo.sensors.xacro" />
+ <!--
+  <xacro:include filename="$(find r2_gazebo)/urdf/gazebo_plugins/p3d_base_controller.xacro" />
   <xacro:include filename="$(find r2_gazebo)/urdf/gazebo_plugins/gazebo_interface.xacro" />
   <xacro:include filename="$(find r2_gazebo)/urdf/gazebo_plugins/leg_grippers.xacro" />

File: r2_gazebo/urdf/sensors/camera.gazebo.xacro (robot description, xacro)
@@ -26,5 +26,5 @@
       </camera>
       <plugin name="camera_controller" filename="libgazebo_ros_camera.so">
-        <alwaysOn>false</alwaysOn>
+        <alwaysOn>0</alwaysOn>
         <updateRate>0.0</updateRate>
         <cameraName>${camera_name}</cameraName>

File: r2_gazebo/urdf/sensors/hokuyo_lx30_laser.gazebo.xacro (robot description, xacro)
@@ -1,10 +1,7 @@
-<?xml version="1.0"?>
-<robot xmlns:sensor="http://playerstage.sourceforge.net/gazebo/xmlschema/#sensor"
-       xmlns:controller="http://playerstage.sourceforge.net/gazebo/xmlschema/#controller"
-       xmlns:interface="http://playerstage.sourceforge.net/gazebo/xmlschema/#interface"
-       xmlns:xacro="http://ros.org/wiki/xacro">
-  <xacro:macro name="hokuyo_lx30_laser_gazebo_v0" params="name ros_topic update_rate min_angle max_angle">
-    <gazebo reference="${name}_link">
-      <sensor:ray name="${name}">
+<?xml version="1.0" ?>
+<robot xmlns:xacro="http://www.ros.org/wiki/xacro" name="r2">
+  <xacro:macro name="hokuyo_lx30_laser_gazebo_v0" params="parent name ros_topic update_rate min_angle max_angle">
+<!--     <gazebo reference="${name}_link">
+      <sensor name="${name}" type="ray">
         <rayCount>640</rayCount>
         <rangeCount>640</rangeCount>
@@ -18,5 +15,5 @@
         <resRange>0.01</resRange>
         <updateRate>${update_rate}</updateRate>
-        <controller:gazebo_ros_laser name="gazebo_ros_${name}_controller" plugin="libgazebo_ros_laser.so">
+        <plugin name="gazebo_ros_${name}_controller" filename="libgazebo_ros_laser.so">
           <gaussianNoise>0.005</gaussianNoise>
           <alwaysOn>true</alwaysOn>
@@ -25,6 +22,31 @@
           <frameName>${name}_link</frameName>
           <interface:laser name="gazebo_ros_${name}_iface" />
-        </controller:gazebo_ros_laser>
-      </sensor:ray>
+        </plugin>
+      </sensor>
+    </gazebo> -->
+  <gazebo reference="${parent}">>
+    <sensor name="${name}" type="ray">
+        <pose>0 0 0 0 0 0</pose>
+    <topic>${ros_topic}</topic>
+        <ray>
+          <scan>
+            <horizontal>
+              <samples>640</samples>
+              <resolution>1</resolution>
+              <min_angle>${min_angle*180.0/3.14159}</min_angle>
+              <max_angle>${max_angle*180.0/3.14159}</max_angle>
+            </horizontal>
+          </scan>
+          <range>
+            <min>0.08</min>
+            <max>10</max>
+            <resolution>0.01</resolution>
+          </range>
+        </ray>
+        <plugin name="laser" filename="libgazebo_ros_laser.so" />
+        <always_on>1</always_on>
+        <update_rate>${update_rate}</update_rate>
+        <visualize>true</visualize>
+      </sensor>
     </gazebo>
   </xacro:macro>

File: r2_gazebo/urdf/sensors/r2.gazebo.sensors.xacro (robot description, xacro)
@@ -4,11 +4,8 @@
 			xmlns:sensor="http://playerstage.sourceforge.net/gazebo/xmlschema/#sensor"
 			xmlns:xacro="http://playerstage.sourceforge.net/gazebo/xmlschema/#interface">
-<!--   <xacro:include filename="$(find r2_gazebo)/urdf/sensors/grasshopper2.gazebo.xacro" />
- -->
  <xacro:include filename="$(find r2_gazebo)/urdf/sensors/asus.gazebo.xacro" />
  <xacro:include filename="$(find r2_gazebo)/urdf/sensors/camera.gazebo.xacro" />
-<!--   <xacro:camera_sensor camera_name="${robot_name}head/camera/left" frame_name="${robot_name}left_camera_optical_frame" />
-  <xacro:camera_sensor camera_name="${robot_name}head/camera/right" frame_name="${robot_name}right_camera_optical_frame" />
- -->
-  <xacro:asus_sensor sensor_name="${robot_name}asus" parent_camera_link="${robot_name}simulated_asus_camera_frame" parent_depth_link="${robot_name}simulated_asus_depth_frame"/>
+ <xacro:camera_sensor camera_name="${robot_name}head/camera/left" frame_name="${robot_name}left_camera_optical_frame" />
+ <xacro:camera_sensor camera_name="${robot_name}head/camera/right" frame_name="${robot_name}right_camera_optical_frame" />
+ <xacro:asus_sensor sensor_name="${robot_name}asus" parent_camera_link="${robot_name}simulated_asus_camera_frame" parent_depth_link="${robot_name}simulated_asus_depth_frame"/>
 </robot>
