Commit message: updated with new controller

File: r2_gazebo/robots/r2.display.urdf.xacro (robot description, xacro)
@@ -5,5 +5,5 @@
 			xmlns:xacro="http://playerstage.sourceforge.net/gazebo/xmlschema/#interface">
   <property name="robot_name" value= "/r2/" />
-  <include filename="$(find r2_description)/robots/r2.urdf.xacro" />
+  <include filename="$(find r2_gazebo)/robots/r2.urdf.xacro" />
   <include filename="$(find r2_gazebo)/urdf/r2.gazebo.xacro" />
   <include filename="$(find r2_gazebo)/urdf/sensors/r2.gazebo.sensors.xacro" />

File: r2_gazebo/robots/r2.sim.urdf.xacro (robot description, xacro)
@@ -5,5 +5,5 @@
 			xmlns:xacro="http://playerstage.sourceforge.net/gazebo/xmlschema/#interface">
   <property name="robot_name" value= "/r2/" />
-  <include filename="$(find r2_description)/robots/r2.urdf.xacro" />
+  <include filename="$(find r2_gazebo)/robots/r2.urdf.xacro" />
   <include filename="$(find r2_gazebo)/urdf/r2.gazebo.xacro" />
   <include filename="$(find r2_gazebo)/urdf/sensors/r2.gazebo.sensors.xacro" />

File: r2_gazebo/robots/r2c_full_body.sim.urdf.xacro (robot description, xacro)
@@ -5,14 +5,20 @@
 			xmlns:xacro="http://playerstage.sourceforge.net/gazebo/xmlschema/#interface">
   <property name="robot_name" value= "/r2/" />
-  <include filename="$(find r2_description)/robots/r2c_full_body_no_world.urdf.xacro" />
-  <xacro:robot_base_origin>
-    <origin rpy="0 3.14159 1.57079" xyz="0.255 0.9 1.365"/>
-<!--    <origin rpy="0 3.14159 3.14159" xyz="0.5 0.7 1.212"/>-->
-  </xacro:robot_base_origin>
+  <link name="world"/>
+  <property name="robot_name" value= "/r2/" />
+  <!--  transforms in first joint don't seem to work properly-->
+  <joint name="${robot_name}fixed/world/world_ref" type="fixed">
+    <parent link="world"/>
+    <child link="${robot_name}world_ref"/>
+    <origin rpy="0 0 0" xyz="0.0 0.0 0.0"/>
+  </joint>
+  <include filename="$(find r2_gazebo)/urdf/models/r2c_full_body_no_world.urdf.xacro" />
+  <xacro:robot_world_origin>
+    <origin rpy="0 0 0" xyz="0.0 0.0 1.5"/>
+  </xacro:robot_world_origin>
   <include filename="$(find r2_gazebo)/urdf/r2.gazebo.xacro" />
   <include filename="$(find r2_gazebo)/urdf/sensors/r2.gazebo.sensors.xacro" />
   <include filename="$(find r2_gazebo)/urdf/r2c_legs.gazebo.xacro" />
   <include filename="$(find r2_gazebo)/urdf/sensors/r2c_legs.gazebo.sensors.xacro" />
-  <include filename="$(find r2_gazebo)/urdf/gazebo_plugins/p3d_base_controller.xacro" />
   <include filename="$(find r2_gazebo)/urdf/gazebo_plugins/gazebo_interface.xacro" />
   <include filename="$(find r2_gazebo)/urdf/gazebo_plugins/leg_grippers.xacro" />

File: r2_gazebo/robots/r2c_legs.display.urdf.xacro (robot description, xacro)
@@ -5,5 +5,5 @@
 			xmlns:xacro="http://playerstage.sourceforge.net/gazebo/xmlschema/#interface">
   <property name="robot_name" value= "/r2/" />
-  <include filename="$(find r2_description)/robots/r2c_legs.urdf.xacro" />
+  <include filename="$(find r2_gazebo)/urdf/models/r2c_legs.urdf.xacro" />
   <include filename="$(find r2_gazebo)/urdf/r2c_legs.gazebo.xacro" />
   <include filename="$(find r2_gazebo)/urdf/sensors/r2c_legs.gazebo.sensors.xacro" />

File: r2_gazebo/robots/r2c_legs.sim.urdf.xacro (robot description, xacro)
@@ -5,5 +5,5 @@
 			xmlns:xacro="http://playerstage.sourceforge.net/gazebo/xmlschema/#interface">
   <property name="robot_name" value= "/r2/" />
-  <include filename="$(find r2_description)/robots/r2c_legs.urdf.xacro" />
+  <include filename="$(find r2_gazebo)/urdf/models/r2c_legs.urdf.xacro" />
   <include filename="$(find r2_gazebo)/urdf/r2c_legs.gazebo.xacro" />
   <include filename="$(find r2_gazebo)/urdf/sensors/r2c_legs.gazebo.sensors.xacro" />

File: r2_gazebo/urdf/gazebo_plugins/gazebo_interface.xacro (robot description, xacro)
@@ -10,5 +10,7 @@
       <jointCommandsTopic>joint_commands</jointCommandsTopic>
       <jointStatesTopic>joint_states</jointStatesTopic>
-      <jointStatesRate>20.0</jointStatesRate> <!--Hz, omit for fastest possible-->
+      <jointCapabilitiesTopic>joint_capabilities</jointCapabilitiesTopic>
+      <jointCommandRefsTopic>joint_command_refs</jointCommandRefsTopic>
+      <jointStatesRate>50.0</jointStatesRate> <!--Hz, omit for fastest possible-->
       <advancedMode>false</advancedMode>
       <!-- if advancedMode=false, joint brakes, etc are not simulated and the following parameters are ignored -->

File: r2_gazebo/urdf/gazebo_plugins/p3d_base_controller.xacro (robot description, xacro)
@@ -7,6 +7,6 @@
     <controller:gazebo_ros_p3d name="p3d_base_controller" plugin="libgazebo_ros_p3d.so">
 <!--      <robotNamespace>r2sim</robotNamespace>-->
-      <bodyName>/r2/robot_base</bodyName>
-      <topicName>/r2/robot_base/pose_state</topicName>
+      <bodyName>/r2/world_ref</bodyName>
+      <topicName>/r2/world_ref/pose_state</topicName>
       <gaussianNoise>0.0</gaussianNoise>
       <frameName>world</frameName>
@@ -15,5 +15,5 @@
       <interface:position name="p3d_base_position"/>
     </controller:gazebo_ros_p3d>
-    <canonicalBody>/r2/robot_world</canonicalBody>
+    <canonicalBody>/r2/world_ref</canonicalBody>
   </gazebo>
 </robot>

File: r2_gazebo/urdf/taskboard.urdf.xacro (robot description, xacro)
@@ -5,5 +5,3 @@
 			xmlns:xacro="http://playerstage.sourceforge.net/gazebo/xmlschema/#interface">
   <include filename="$(find r2_gazebo)/urdf/taskboard.lower.xacro" />
-  <include filename="$(find r2_gazebo)/urdf/gazebo_plugins/gazebo_interface.xacro" />
-  <include filename="$(find r2_gazebo)/urdf/gazebo_plugins/taskboard.panel_a.controller.xacro" />
- </robot>
+</robot>
