Commit message: One model for taskboard

File: r2_gazebo/urdf/taskboard.B01.xacro (robot description, xacro)
@@ -1,38 +1,6 @@
 <?xml version="1.0"?>
-<robot>
-  <link name="world"/>
-  <link name="dummy">
-    <inertial>
-      <mass value="1"/>
-      <inertia ixx="1" ixy="0.0" ixz="0.0" iyy="1" iyz="0.0" izz="1"/>
-    </inertial>
-  </link>
-  <link name="Taskboard">
-    <inertial>
-      <mass value="1"/>
-      <inertia ixx="1" ixy="0.0" ixz="0.0" iyy="1" iyz="0.0" izz="1"/>
-    </inertial>
-  </link>
-  <link name="Taskboard_Slot2">
-    <inertial>
-      <mass value="1"/>
-      <inertia ixx="1" ixy="0.0" ixz="0.0" iyy="1" iyz="0.0" izz="1"/>
-    </inertial>
-  </link>
-<!--
-  <link name="Link1_X">
-    <inertial>
-      <mass value=".01"/>
-      <inertia ixx="1" ixy="0.0" ixz="0.0" iyy="1" iyz="0.0" izz="1"/>
-    </inertial>
-  </link>
-  <link name="Link1_Y">
-    <inertial>
-      <mass value=".01"/>
-      <inertia ixx="1" ixy="0.0" ixz="0.0" iyy="1" iyz="0.0" izz="1"/>
-    </inertial>
-  </link>
--->
-  <link name="Link1">
+<robot xmlns:xacro="http://www.ros.org/wiki/xacro" name="taskboard_B01">
+  <xacro:property name="prefix" value="taskboard_b01_" />
+  <link name="${prefix}Link1">
     <visual>
       <geometry>
@@ -52,17 +20,17 @@
     </inertial>
   </link>
-  <link name="Link2_X">
-    <inertial>
-      <mass value=".01"/>
-      <inertia ixx="1" ixy="0.0" ixz="0.0" iyy="1" iyz="0.0" izz="1"/>
-    </inertial>
-  </link>
-  <link name="Link2_Y">
-    <inertial>
-      <mass value=".01"/>
-      <inertia ixx="1" ixy="0.0" ixz="0.0" iyy="1" iyz="0.0" izz="1"/>
-    </inertial>
-  </link>
-  <link name="Link2">
+  <link name="${prefix}Link2_X">
+    <inertial>
+      <mass value=".01"/>
+      <inertia ixx="1" ixy="0.0" ixz="0.0" iyy="1" iyz="0.0" izz="1"/>
+    </inertial>
+  </link>
+  <link name="${prefix}Link2_Y">
+    <inertial>
+      <mass value=".01"/>
+      <inertia ixx="1" ixy="0.0" ixz="0.0" iyy="1" iyz="0.0" izz="1"/>
+    </inertial>
+  </link>
+  <link name="${prefix}Link2">
     <visual>
       <geometry>
@@ -82,17 +50,17 @@
     </inertial>
   </link>
-  <link name="Link3_X">
-    <inertial>
-      <mass value=".01"/>
-      <inertia ixx="1" ixy="0.0" ixz="0.0" iyy="1" iyz="0.0" izz="1"/>
-    </inertial>
-  </link>
-  <link name="Link3_Y">
-    <inertial>
-      <mass value=".01"/>
-      <inertia ixx="1" ixy="0.0" ixz="0.0" iyy="1" iyz="0.0" izz="1"/>
-    </inertial>
-  </link>
-  <link name="Link3">
+  <link name="${prefix}Link3_X">
+    <inertial>
+      <mass value=".01"/>
+      <inertia ixx="1" ixy="0.0" ixz="0.0" iyy="1" iyz="0.0" izz="1"/>
+    </inertial>
+  </link>
+  <link name="${prefix}Link3_Y">
+    <inertial>
+      <mass value=".01"/>
+      <inertia ixx="1" ixy="0.0" ixz="0.0" iyy="1" iyz="0.0" izz="1"/>
+    </inertial>
+  </link>
+  <link name="${prefix}Link3">
     <visual>
       <geometry>
@@ -112,17 +80,17 @@
     </inertial>
   </link>
-  <link name="Link4_X">
-    <inertial>
-      <mass value=".01"/>
-      <inertia ixx="1" ixy="0.0" ixz="0.0" iyy="1" iyz="0.0" izz="1"/>
-    </inertial>
-  </link>
-  <link name="Link4_Y">
-    <inertial>
-      <mass value=".01"/>
-      <inertia ixx="1" ixy="0.0" ixz="0.0" iyy="1" iyz="0.0" izz="1"/>
-    </inertial>
-  </link>
-  <link name="Link4">
+  <link name="${prefix}Link4_X">
+    <inertial>
+      <mass value=".01"/>
+      <inertia ixx="1" ixy="0.0" ixz="0.0" iyy="1" iyz="0.0" izz="1"/>
+    </inertial>
+  </link>
+  <link name="${prefix}Link4_Y">
+    <inertial>
+      <mass value=".01"/>
+      <inertia ixx="1" ixy="0.0" ixz="0.0" iyy="1" iyz="0.0" izz="1"/>
+    </inertial>
+  </link>
+  <link name="${prefix}Link4">
     <visual>
       <geometry>
@@ -142,17 +110,17 @@
     </inertial>
   </link>
-  <link name="Link5_X">
-    <inertial>
-      <mass value=".01"/>
-      <inertia ixx="1" ixy="0.0" ixz="0.0" iyy="1" iyz="0.0" izz="1"/>
-    </inertial>
-  </link>
-  <link name="Link5_Y">
-    <inertial>
-      <mass value=".01"/>
-      <inertia ixx="1" ixy="0.0" ixz="0.0" iyy="1" iyz="0.0" izz="1"/>
-    </inertial>
-  </link>
-  <link name="Link5">
+  <link name="${prefix}Link5_X">
+    <inertial>
+      <mass value=".01"/>
+      <inertia ixx="1" ixy="0.0" ixz="0.0" iyy="1" iyz="0.0" izz="1"/>
+    </inertial>
+  </link>
+  <link name="${prefix}Link5_Y">
+    <inertial>
+      <mass value=".01"/>
+      <inertia ixx="1" ixy="0.0" ixz="0.0" iyy="1" iyz="0.0" izz="1"/>
+    </inertial>
+  </link>
+  <link name="${prefix}Link5">
     <visual>
       <geometry>
@@ -172,17 +140,17 @@
     </inertial>
   </link>
-  <link name="Taskboard_Slot2_B01_X">
-    <inertial>
-      <mass value=".01"/>
-      <inertia ixx="1" ixy="0.0" ixz="0.0" iyy="1" iyz="0.0" izz="1"/>
-    </inertial>
-  </link>
-  <link name="Taskboard_Slot2_B01_Y">
-    <inertial>
-      <mass value=".01"/>
-      <inertia ixx="1" ixy="0.0" ixz="0.0" iyy="1" iyz="0.0" izz="1"/>
-    </inertial>
-  </link>
-  <link name="Taskboard_Slot2_B01">
+  <link name="${prefix}Taskboard_Slot2_B01_X">
+    <inertial>
+      <mass value=".01"/>
+      <inertia ixx="1" ixy="0.0" ixz="0.0" iyy="1" iyz="0.0" izz="1"/>
+    </inertial>
+  </link>
+  <link name="${prefix}Taskboard_Slot2_B01_Y">
+    <inertial>
+      <mass value=".01"/>
+      <inertia ixx="1" ixy="0.0" ixz="0.0" iyy="1" iyz="0.0" izz="1"/>
+    </inertial>
+  </link>
+  <link name="${prefix}Taskboard_Slot2_B01">
     <visual>
       <geometry>
@@ -202,48 +170,15 @@
     </inertial>
   </link>
-  <joint name="world/dummy" type="fixed">
-    <parent link="world"/>
-    <child link="dummy"/>
-    <origin rpy="0.0 0 0" xyz="0.0 0.0 0.0"/>
-  </joint>
-  <joint name="dummy/Taskboard" type="fixed">
-    <parent link="dummy"/>
-    <child link="Taskboard"/>
-    <origin rpy="1.57 0 3.14" xyz=".02 -.48 1.3"/>
-  </joint>
-  <joint name="Taskboard/Taskboard_slot2" type="fixed">
-    <parent link="Taskboard"/>
-    <child link="Taskboard_Slot2"/>
-    <origin rpy="0 0 0" xyz="-0.121 0 0"/>
-  </joint>
-<!--
-  <joint name="Taskboard_Slot2/Link1_X" type="continuous">
-    <parent link="Taskboard_Slot2"/>
-    <child link="Link1_X"/>
+  <joint name="${prefix}Taskboard_Slot2/Link1" type="continuous">
+    <parent link="taskboard_slot2"/>
+    <child link="${prefix}Link1"/>
     <origin rpy="0 0 0" xyz="0 0.09195 0.01746"/>
-    <axis xyz="1 0 0"/>
-    <limit effort="100" velocity="100"/>
-    <dynamics damping=".1" friction=".1" />
-  </joint>
-  <joint name="Link1_X/Link1_Y" type="continuous">
-    <parent link="Link1_X"/>
-    <child link="Link1_Y"/>
-    <origin rpy="0 0 0" xyz="0 0 0"/>
-    <axis xyz="0 1 0"/>
-    <limit effort="100" velocity="100"/>
-    <dynamics damping=".1" friction=".1" />
-  </joint>
--->
-  <joint name="Taskboard_Slot2/Link1" type="continuous">
-    <parent link="Taskboard_Slot2"/>
-    <child link="Link1"/>
-    <origin rpy="0 0 0" xyz="0 0.09195 0.01746"/>
-    <axis xyz="0 0 1"/>
-    <limit effort="100" velocity="100"/>
-    <dynamics damping=".1" friction=".1" />
-  </joint>
-  <joint name="Link1/Link2_X" type="continuous">
-    <parent link="Link1"/>
-    <child link="Link2_X"/>
+    <axis xyz="0 0 1"/>
+    <limit effort="100" velocity="100"/>
+    <dynamics damping=".1" friction=".1" />
+  </joint>
+  <joint name="${prefix}Link1/Link2_X" type="continuous">
+    <parent link="${prefix}Link1"/>
+    <child link="${prefix}Link2_X"/>
     <origin rpy="0 0 0" xyz="0 0 0.066"/>
     <axis xyz="1 0 0"/>
@@ -251,15 +186,15 @@
     <dynamics damping=".1" friction=".1" />
   </joint>
-  <joint name="Link2_X/Link2_Y" type="continuous">
-    <parent link="Link2_X"/>
-    <child link="Link2_Y"/>
-    <origin rpy="0 0 0" xyz="0 0 0"/>
-    <axis xyz="0 1 0"/>
-    <limit effort="100" velocity="100"/>
-    <dynamics damping=".1" friction=".1" />
-  </joint>
-  <joint name="Link2_Y/Link2" type="continuous">
-    <parent link="Link2_Y"/>
-    <child link="Link2"/>
+  <joint name="${prefix}Link2_X/Link2_Y" type="continuous">
+    <parent link="${prefix}Link2_X"/>
+    <child link="${prefix}Link2_Y"/>
+    <origin rpy="0 0 0" xyz="0 0 0"/>
+    <axis xyz="0 1 0"/>
+    <limit effort="100" velocity="100"/>
+    <dynamics damping=".1" friction=".1" />
+  </joint>
+  <joint name="${prefix}Link2_Y/Link2" type="continuous">
+    <parent link="${prefix}Link2_Y"/>
+    <child link="${prefix}Link2"/>
     <origin rpy="1.5708 0 0" xyz="0 0 0"/>
     <axis xyz="0 0 1"/>
@@ -267,7 +202,7 @@
     <dynamics damping=".1" friction=".1" />
   </joint>
-  <joint name="Link2/Link3_X" type="continuous">
-    <parent link="Link2"/>
-    <child link="Link3_X"/>
+  <joint name="${prefix}Link2/Link3_X" type="continuous">
+    <parent link="${prefix}Link2"/>
+    <child link="${prefix}Link3_X"/>
     <origin rpy="0 0 0" xyz="0 0 0.04033"/>
     <axis xyz="1 0 0"/>
@@ -275,23 +210,23 @@
     <dynamics damping=".1" friction=".1" />
   </joint>
-  <joint name="Link3_X/Link3_Y" type="continuous">
-    <parent link="Link3_X"/>
-    <child link="Link3_Y"/>
-    <origin rpy="0 0 0" xyz="0 0 0"/>
-    <axis xyz="0 1 0"/>
-    <limit effort="100" velocity="100"/>
-    <dynamics damping=".1" friction=".1" />
-  </joint>
-  <joint name="Link3_Y/Link3" type="continuous">
-    <parent link="Link3_Y"/>
-    <child link="Link3"/>
-    <origin rpy="0 0 0" xyz="0 0 0"/>
-    <axis xyz="0 0 1"/>
-    <limit effort="100" velocity="100"/>
-    <dynamics damping=".1" friction=".1" />
-  </joint>
-  <joint name="Link3/Link4_X" type="continuous">
-    <parent link="Link3"/>
-    <child link="Link4_X"/>
+  <joint name="${prefix}Link3_X/Link3_Y" type="continuous">
+    <parent link="${prefix}Link3_X"/>
+    <child link="${prefix}Link3_Y"/>
+    <origin rpy="0 0 0" xyz="0 0 0"/>
+    <axis xyz="0 1 0"/>
+    <limit effort="100" velocity="100"/>
+    <dynamics damping=".1" friction=".1" />
+  </joint>
+  <joint name="${prefix}Link3_Y/Link3" type="continuous">
+    <parent link="${prefix}Link3_Y"/>
+    <child link="${prefix}Link3"/>
+    <origin rpy="0 0 0" xyz="0 0 0"/>
+    <axis xyz="0 0 1"/>
+    <limit effort="100" velocity="100"/>
+    <dynamics damping=".1" friction=".1" />
+  </joint>
+  <joint name="${prefix}Link3/Link4_X" type="continuous">
+    <parent link="${prefix}Link3"/>
+    <child link="${prefix}Link4_X"/>
     <origin rpy="0 0 0" xyz="0 0 0.04733"/>
     <axis xyz="1 0 0"/>
@@ -299,23 +234,23 @@
     <dynamics damping=".1" friction=".1" />
   </joint>
-  <joint name="Link4_X/Link4_Y" type="continuous">
-    <parent link="Link4_X"/>
-    <child link="Link4_Y"/>
-    <origin rpy="0 0 0" xyz="0 0 0"/>
-    <axis xyz="0 1 0"/>
-    <limit effort="100" velocity="100"/>
-    <dynamics damping=".1" friction=".1" />
-  </joint>
-  <joint name="Link4_Y/Link4" type="continuous">
-    <parent link="Link4_Y"/>
-    <child link="Link4"/>
-    <origin rpy="0 0 0" xyz="0 0 0"/>
-    <axis xyz="0 0 1"/>
-    <limit effort="100" velocity="100"/>
-    <dynamics damping=".1" friction=".1" />
-  </joint>
-  <joint name="Link4/Link5_X" type="continuous">
-    <parent link="Link4"/>
-    <child link="Link5_X"/>
+  <joint name="${prefix}Link4_X/Link4_Y" type="continuous">
+    <parent link="${prefix}Link4_X"/>
+    <child link="${prefix}Link4_Y"/>
+    <origin rpy="0 0 0" xyz="0 0 0"/>
+    <axis xyz="0 1 0"/>
+    <limit effort="100" velocity="100"/>
+    <dynamics damping=".1" friction=".1" />
+  </joint>
+  <joint name="${prefix}Link4_Y/Link4" type="continuous">
+    <parent link="${prefix}Link4_Y"/>
+    <child link="${prefix}Link4"/>
+    <origin rpy="0 0 0" xyz="0 0 0"/>
+    <axis xyz="0 0 1"/>
+    <limit effort="100" velocity="100"/>
+    <dynamics damping=".1" friction=".1" />
+  </joint>
+  <joint name="${prefix}Link4/Link5_X" type="continuous">
+    <parent link="${prefix}Link4"/>
+    <child link="${prefix}Link5_X"/>
     <origin rpy="0 0 0" xyz="0 0 0.03811"/>
     <axis xyz="1 0 0"/>
@@ -323,15 +258,15 @@
     <dynamics damping=".1" friction=".1" />
   </joint>
-  <joint name="Link5_X/Link5_Y" type="continuous">
-    <parent link="Link5_X"/>
-    <child link="Link5_Y"/>
-    <origin rpy="0 0 0" xyz="0 0 0"/>
-    <axis xyz="0 1 0"/>
-    <limit effort="100" velocity="100"/>
-    <dynamics damping=".1" friction=".1" />
-  </joint>
-  <joint name="Link5_Y/Link5" type="continuous">
-    <parent link="Link5_Y"/>
-    <child link="Link5"/>
+  <joint name="${prefix}Link5_X/Link5_Y" type="continuous">
+    <parent link="${prefix}Link5_X"/>
+    <child link="${prefix}Link5_Y"/>
+    <origin rpy="0 0 0" xyz="0 0 0"/>
+    <axis xyz="0 1 0"/>
+    <limit effort="100" velocity="100"/>
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