Commit message: One model for taskboard

File: r2_gazebo/urdf/taskboard.B05.xacro (robot description, xacro)
@@ -1,38 +1,6 @@
 <?xml version="1.0"?>
-<robot>
-  <link name="world"/>
-  <link name="dummy">
-    <inertial>
-      <mass value="1"/>
-      <inertia ixx="1" ixy="0.0" ixz="0.0" iyy="1" iyz="0.0" izz="1"/>
-    </inertial>
-  </link>
-  <link name="Taskboard">
-    <inertial>
-      <mass value="1"/>
-      <inertia ixx="1" ixy="0.0" ixz="0.0" iyy="1" iyz="0.0" izz="1"/>
-    </inertial>
-  </link>
-  <link name="Taskboard_Slot2">
-    <inertial>
-      <mass value="1"/>
-      <inertia ixx="1" ixy="0.0" ixz="0.0" iyy="1" iyz="0.0" izz="1"/>
-    </inertial>
-  </link>
-<!--
-  <link name="Link1_X">
-    <inertial>
-      <mass value=".01"/>
-      <inertia ixx="1" ixy="0.0" ixz="0.0" iyy="1" iyz="0.0" izz="1"/>
-    </inertial>
-  </link>
-  <link name="Link1_Y">
-    <inertial>
-      <mass value=".01"/>
-      <inertia ixx="1" ixy="0.0" ixz="0.0" iyy="1" iyz="0.0" izz="1"/>
-    </inertial>
-  </link>
--->
-  <link name="Link1">
+<robot xmlns:xacro="http://www.ros.org/wiki/xacro" name="taskboard_B05">
+  <xacro:property name="b5prefix" value="taskboard_b05_" />
+  <link name="${b5prefix}Link1">
     <visual>
       <geometry>
@@ -52,17 +20,17 @@
     </inertial>
   </link>
-  <link name="Link2_X">
-    <inertial>
-      <mass value=".01"/>
-      <inertia ixx="1" ixy="0.0" ixz="0.0" iyy="1" iyz="0.0" izz="1"/>
-    </inertial>
-  </link>
-  <link name="Link2_Y">
-    <inertial>
-      <mass value=".01"/>
-      <inertia ixx="1" ixy="0.0" ixz="0.0" iyy="1" iyz="0.0" izz="1"/>
-    </inertial>
-  </link>
-  <link name="Link2">
+  <link name="${b5prefix}Link2_X">
+    <inertial>
+      <mass value=".01"/>
+      <inertia ixx="1" ixy="0.0" ixz="0.0" iyy="1" iyz="0.0" izz="1"/>
+    </inertial>
+  </link>
+  <link name="${b5prefix}Link2_Y">
+    <inertial>
+      <mass value=".01"/>
+      <inertia ixx="1" ixy="0.0" ixz="0.0" iyy="1" iyz="0.0" izz="1"/>
+    </inertial>
+  </link>
+  <link name="${b5prefix}Link2">
     <visual>
       <geometry>
@@ -82,17 +50,17 @@
     </inertial>
   </link>
-  <link name="Link3_X">
-    <inertial>
-      <mass value=".01"/>
-      <inertia ixx="1" ixy="0.0" ixz="0.0" iyy="1" iyz="0.0" izz="1"/>
-    </inertial>
-  </link>
-  <link name="Link3_Y">
-    <inertial>
-      <mass value=".01"/>
-      <inertia ixx="1" ixy="0.0" ixz="0.0" iyy="1" iyz="0.0" izz="1"/>
-    </inertial>
-  </link>
-  <link name="Link3">
+  <link name="${b5prefix}Link3_X">
+    <inertial>
+      <mass value=".01"/>
+      <inertia ixx="1" ixy="0.0" ixz="0.0" iyy="1" iyz="0.0" izz="1"/>
+    </inertial>
+  </link>
+  <link name="${b5prefix}Link3_Y">
+    <inertial>
+      <mass value=".01"/>
+      <inertia ixx="1" ixy="0.0" ixz="0.0" iyy="1" iyz="0.0" izz="1"/>
+    </inertial>
+  </link>
+  <link name="${b5prefix}Link3">
     <visual>
       <geometry>
@@ -112,17 +80,17 @@
     </inertial>
   </link>
-  <link name="Link4_X">
-    <inertial>
-      <mass value=".01"/>
-      <inertia ixx="1" ixy="0.0" ixz="0.0" iyy="1" iyz="0.0" izz="1"/>
-    </inertial>
-  </link>
-  <link name="Link4_Y">
-    <inertial>
-      <mass value=".01"/>
-      <inertia ixx="1" ixy="0.0" ixz="0.0" iyy="1" iyz="0.0" izz="1"/>
-    </inertial>
-  </link>
-  <link name="Link4">
+  <link name="${b5prefix}Link4_X">
+    <inertial>
+      <mass value=".01"/>
+      <inertia ixx="1" ixy="0.0" ixz="0.0" iyy="1" iyz="0.0" izz="1"/>
+    </inertial>
+  </link>
+  <link name="${b5prefix}Link4_Y">
+    <inertial>
+      <mass value=".01"/>
+      <inertia ixx="1" ixy="0.0" ixz="0.0" iyy="1" iyz="0.0" izz="1"/>
+    </inertial>
+  </link>
+  <link name="${b5prefix}Link4">
     <visual>
       <geometry>
@@ -142,17 +110,17 @@
     </inertial>
   </link>
-  <link name="Link5_X">
-    <inertial>
-      <mass value=".01"/>
-      <inertia ixx="1" ixy="0.0" ixz="0.0" iyy="1" iyz="0.0" izz="1"/>
-    </inertial>
-  </link>
-  <link name="Link5_Y">
-    <inertial>
-      <mass value=".01"/>
-      <inertia ixx="1" ixy="0.0" ixz="0.0" iyy="1" iyz="0.0" izz="1"/>
-    </inertial>
-  </link>
-  <link name="Link5">
+  <link name="${b5prefix}Link5_X">
+    <inertial>
+      <mass value=".01"/>
+      <inertia ixx="1" ixy="0.0" ixz="0.0" iyy="1" iyz="0.0" izz="1"/>
+    </inertial>
+  </link>
+  <link name="${b5prefix}Link5_Y">
+    <inertial>
+      <mass value=".01"/>
+      <inertia ixx="1" ixy="0.0" ixz="0.0" iyy="1" iyz="0.0" izz="1"/>
+    </inertial>
+  </link>
+  <link name="${b5prefix}Link5">
     <visual>
       <geometry>
@@ -172,17 +140,17 @@
     </inertial>
   </link>
-  <link name="Taskboard_Slot2_B05_X">
-    <inertial>
-      <mass value=".01"/>
-      <inertia ixx="1" ixy="0.0" ixz="0.0" iyy="1" iyz="0.0" izz="1"/>
-    </inertial>
-  </link>
-  <link name="Taskboard_Slot2_B05_Y">
-    <inertial>
-      <mass value=".01"/>
-      <inertia ixx="1" ixy="0.0" ixz="0.0" iyy="1" iyz="0.0" izz="1"/>
-    </inertial>
-  </link>
-  <link name="Taskboard_Slot2_B05">
+  <link name="${b5prefix}Taskboard_Slot2_B05_X">
+    <inertial>
+      <mass value=".01"/>
+      <inertia ixx="1" ixy="0.0" ixz="0.0" iyy="1" iyz="0.0" izz="1"/>
+    </inertial>
+  </link>
+  <link name="${b5prefix}Taskboard_Slot2_B05_Y">
+    <inertial>
+      <mass value=".01"/>
+      <inertia ixx="1" ixy="0.0" ixz="0.0" iyy="1" iyz="0.0" izz="1"/>
+    </inertial>
+  </link>
+  <link name="${b5prefix}Taskboard_Slot2_B05">
     <visual>
       <geometry>
@@ -202,40 +170,7 @@
     </inertial>
   </link>
-  <joint name="world/dummy" type="fixed">
-    <parent link="world"/>
-    <child link="dummy"/>
-    <origin rpy="0.0 0 0" xyz="0.0 0.0 0.0"/>
-  </joint>
-  <joint name="dummy/Taskboard" type="fixed">
-    <parent link="dummy"/>
-    <child link="Taskboard"/>
-    <origin rpy="1.57 0 3.14" xyz=".02 -.48 1.3"/>
-  </joint>
-  <joint name="Taskboard/Taskboard_slot2" type="fixed">
-    <parent link="Taskboard"/>
-    <child link="Taskboard_Slot2"/>
-    <origin rpy="0 0 0" xyz="-0.121 0 0"/>
-  </joint>
-<!--
-  <joint name="Taskboard_Slot2/Link1_X" type="continuous">
-    <parent link="Taskboard_Slot2"/>
-    <child link="Link1_X"/>
-    <origin rpy="0 0 0" xyz="0 0.09195 0.01746"/>
-    <axis xyz="1 0 0"/>
-    <limit effort="100" velocity="100"/>
-    <dynamics damping=".1" friction=".1" />
-  </joint>
-  <joint name="Link1_X/Link1_Y" type="continuous">
-    <parent link="Link1_X"/>
-    <child link="Link1_Y"/>
-    <origin rpy="0 0 0" xyz="0 0 0"/>
-    <axis xyz="0 1 0"/>
-    <limit effort="100" velocity="100"/>
-    <dynamics damping=".1" friction=".1" />
-  </joint>
--->
-  <joint name="Taskboard_Slot2/Link1" type="continuous">
-    <parent link="Taskboard_Slot2"/>
-    <child link="Link1"/>
+  <joint name="${b5prefix}Taskboard_Slot2/Link1" type="continuous">
+    <parent link="taskboard_slot2"/>
+    <child link="${b5prefix}Link1"/>
     <origin rpy="0 0 0" xyz="0 -0.1236 0.01746"/>
     <axis xyz="0 0 1"/>
@@ -243,7 +178,7 @@
     <dynamics damping=".1" friction=".1" />
   </joint>
-  <joint name="Link1/Link2_X" type="continuous">
-    <parent link="Link1"/>
-    <child link="Link2_X"/>
+  <joint name="${b5prefix}Link1/Link2_X" type="continuous">
+    <parent link="${b5prefix}Link1"/>
+    <child link="${b5prefix}Link2_X"/>
     <origin rpy="0 0 0" xyz="0 0 0.066"/>
     <axis xyz="1 0 0"/>
@@ -251,15 +186,15 @@
     <dynamics damping=".1" friction=".1" />
   </joint>
-  <joint name="Link2_X/Link2_Y" type="continuous">
-    <parent link="Link2_X"/>
-    <child link="Link2_Y"/>
-    <origin rpy="0 0 0" xyz="0 0 0"/>
-    <axis xyz="0 1 0"/>
-    <limit effort="100" velocity="100"/>
-    <dynamics damping=".1" friction=".1" />
-  </joint>
-  <joint name="Link2_Y/Link2" type="continuous">
-    <parent link="Link2_Y"/>
-    <child link="Link2"/>
+  <joint name="${b5prefix}Link2_X/Link2_Y" type="continuous">
+    <parent link="${b5prefix}Link2_X"/>
+    <child link="${b5prefix}Link2_Y"/>
+    <origin rpy="0 0 0" xyz="0 0 0"/>
+    <axis xyz="0 1 0"/>
+    <limit effort="100" velocity="100"/>
+    <dynamics damping=".1" friction=".1" />
+  </joint>
+  <joint name="${b5prefix}Link2_Y/Link2" type="continuous">
+    <parent link="${b5prefix}Link2_Y"/>
+    <child link="${b5prefix}Link2"/>
     <origin rpy="1.5708 0 0" xyz="0 0 0"/>
     <axis xyz="0 0 1"/>
@@ -267,7 +202,7 @@
     <dynamics damping=".1" friction=".1" />
   </joint>
-  <joint name="Link2/Link3_X" type="continuous">
-    <parent link="Link2"/>
-    <child link="Link3_X"/>
+  <joint name="${b5prefix}Link2/Link3_X" type="continuous">
+    <parent link="${b5prefix}Link2"/>
+    <child link="${b5prefix}Link3_X"/>
     <origin rpy="0 0 0" xyz="0 0 0.04033"/>
     <axis xyz="1 0 0"/>
@@ -275,23 +210,23 @@
     <dynamics damping=".1" friction=".1" />
   </joint>
-  <joint name="Link3_X/Link3_Y" type="continuous">
-    <parent link="Link3_X"/>
-    <child link="Link3_Y"/>
-    <origin rpy="0 0 0" xyz="0 0 0"/>
-    <axis xyz="0 1 0"/>
-    <limit effort="100" velocity="100"/>
-    <dynamics damping=".1" friction=".1" />
-  </joint>
-  <joint name="Link3_Y/Link3" type="continuous">
-    <parent link="Link3_Y"/>
-    <child link="Link3"/>
-    <origin rpy="0 0 0" xyz="0 0 0"/>
-    <axis xyz="0 0 1"/>
-    <limit effort="100" velocity="100"/>
-    <dynamics damping=".1" friction=".1" />
-  </joint>
-  <joint name="Link3/Link4_X" type="continuous">
-    <parent link="Link3"/>
-    <child link="Link4_X"/>
+  <joint name="${b5prefix}Link3_X/Link3_Y" type="continuous">
+    <parent link="${b5prefix}Link3_X"/>
+    <child link="${b5prefix}Link3_Y"/>
+    <origin rpy="0 0 0" xyz="0 0 0"/>
+    <axis xyz="0 1 0"/>
+    <limit effort="100" velocity="100"/>
+    <dynamics damping=".1" friction=".1" />
+  </joint>
+  <joint name="${b5prefix}Link3_Y/Link3" type="continuous">
+    <parent link="${b5prefix}Link3_Y"/>
+    <child link="${b5prefix}Link3"/>
+    <origin rpy="0 0 0" xyz="0 0 0"/>
+    <axis xyz="0 0 1"/>
+    <limit effort="100" velocity="100"/>
+    <dynamics damping=".1" friction=".1" />
+  </joint>
+  <joint name="${b5prefix}Link3/Link4_X" type="continuous">
+    <parent link="${b5prefix}Link3"/>
+    <child link="${b5prefix}Link4_X"/>
     <origin rpy="0 0 0" xyz="0 0 0.04733"/>
     <axis xyz="1 0 0"/>
@@ -299,23 +234,23 @@
     <dynamics damping=".1" friction=".1" />
   </joint>
-  <joint name="Link4_X/Link4_Y" type="continuous">
-    <parent link="Link4_X"/>
-    <child link="Link4_Y"/>
-    <origin rpy="0 0 0" xyz="0 0 0"/>
-    <axis xyz="0 1 0"/>
-    <limit effort="100" velocity="100"/>
-    <dynamics damping=".1" friction=".1" />
-  </joint>
-  <joint name="Link4_Y/Link4" type="continuous">
-    <parent link="Link4_Y"/>
-    <child link="Link4"/>
-    <origin rpy="0 0 0" xyz="0 0 0"/>
-    <axis xyz="0 0 1"/>
-    <limit effort="100" velocity="100"/>
-    <dynamics damping=".1" friction=".1" />
-  </joint>
-  <joint name="Link4/Link5_X" type="continuous">
-    <parent link="Link4"/>
-    <child link="Link5_X"/>
+  <joint name="${b5prefix}Link4_X/Link4_Y" type="continuous">
+    <parent link="${b5prefix}Link4_X"/>
+    <child link="${b5prefix}Link4_Y"/>
+    <origin rpy="0 0 0" xyz="0 0 0"/>
+    <axis xyz="0 1 0"/>
+    <limit effort="100" velocity="100"/>
+    <dynamics damping=".1" friction=".1" />
+  </joint>
+  <joint name="${b5prefix}Link4_Y/Link4" type="continuous">
+    <parent link="${b5prefix}Link4_Y"/>
+    <child link="${b5prefix}Link4"/>
+    <origin rpy="0 0 0" xyz="0 0 0"/>
+    <axis xyz="0 0 1"/>
+    <limit effort="100" velocity="100"/>
+    <dynamics damping=".1" friction=".1" />
+  </joint>
+  <joint name="${b5prefix}Link4/Link5_X" type="continuous">
+    <parent link="${b5prefix}Link4"/>
+    <child link="${b5prefix}Link5_X"/>
     <origin rpy="0 0 0" xyz="0 0 0.03811"/>
     <axis xyz="1 0 0"/>
@@ -323,15 +258,15 @@
     <dynamics damping=".1" friction=".1" />
   </joint>
-  <joint name="Link5_X/Link5_Y" type="continuous">
-    <parent link="Link5_X"/>
-    <child link="Link5_Y"/>
-    <origin rpy="0 0 0" xyz="0 0 0"/>
-    <axis xyz="0 1 0"/>
-    <limit effort="100" velocity="100"/>
-    <dynamics damping=".1" friction=".1" />
-  </joint>
-  <joint name="Link5_Y/Link5" type="continuous">
-    <parent link="Link5_Y"/>
-    <child link="Link5"/>
+  <joint name="${b5prefix}Link5_X/Link5_Y" type="continuous">
+    <parent link="${b5prefix}Link5_X"/>
+    <child link="${b5prefix}Link5_Y"/>
+    <origin rpy="0 0 0" xyz="0 0 0"/>
+    <axis xyz="0 1 0"/>
+    <limit effort="100" velocity="100"/>
+    <dynamics damping=".1" friction=".1" />
+  </joint>
+  <joint name="${b5prefix}Link5_Y/Link5" type="continuous">
+    <parent link="${b5prefix}Link5_Y"/>
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
File: r2_gazebo/urdf/taskboard.urdf.xacro (robot description, xacro)
@@ -2,4 +2,6 @@
 <robot name="taskboard" xmlns:xacro="http://wiki.ros.org/xacro">
   <xacro:include filename="$(find r2_gazebo)/urdf/taskboard.lower.xacro" />
+  <xacro:include filename="$(find r2_gazebo)/urdf/taskboard.B01.xacro" />
+  <xacro:include filename="$(find r2_gazebo)/urdf/taskboard.B05.xacro" />
   <xacro:include filename="$(find r2_gazebo)/urdf/gazebo_plugins/gazebo_interface.xacro" />
   <xacro:include filename="$(find r2_gazebo)/urdf/gazebo_plugins/taskboard.panel_a.controller.xacro" />
