Commit message: modified taskboard to add pullouts to lower switches

File: r2_gazebo/urdf/taskboard.lower.xacro (robot description, xacro)
@@ -224,4 +224,10 @@
     </inertial>
   </link>
+  <link name="taskboard_slot1_switch2_pullout">
+    <inertial>
+      <mass value=".01"/>
+      <inertia ixx="1" ixy="0.0" ixz="0.0" iyy="1" iyz="0.0" izz="1"/>
+    </inertial>
+  </link>
   <link name="taskboard_slot1_switch2">
     <visual>
@@ -242,4 +248,10 @@
     </inertial>
   </link>
+  <link name="taskboard_slot1_switch3_pullout">
+    <inertial>
+      <mass value=".01"/>
+      <inertia ixx="1" ixy="0.0" ixz="0.0" iyy="1" iyz="0.0" izz="1"/>
+    </inertial>
+  </link>
   <link name="taskboard_slot1_switch3">
     <visual>
@@ -257,4 +269,10 @@
     <inertial>
       <mass value="5"/>
+      <inertia ixx="1" ixy="0.0" ixz="0.0" iyy="1" iyz="0.0" izz="1"/>
+    </inertial>
+  </link>
+  <link name="taskboard_slot1_switch4_pullout">
+    <inertial>
+      <mass value=".01"/>
       <inertia ixx="1" ixy="0.0" ixz="0.0" iyy="1" iyz="0.0" izz="1"/>
     </inertial>
@@ -881,22 +899,43 @@
   <joint name="taskboard_lower/taskboard_slot1_switch2" type="revolute">
     <parent link="taskboard_slot1"/>
-    <child link="taskboard_slot1_switch2"/>
+    <child link="taskboard_slot1_switch2_pullout"/>
     <origin rpy=".47 0 0" xyz="-.0635 -.089 0.009"/>
     <axis xyz="1 0 0"/>
     <limit effort="10000000.0" lower="-.94" upper="0" velocity="1000"/>
   </joint>
+  <joint name="taskboard_lower/taskboard_slot1_switch2_pullout" type="prismatic">
+    <parent link="taskboard_slot1_switch2_pullout"/>
+    <child link="taskboard_slot1_switch2"/>
+    <origin rpy="0 0 0" xyz="0 0 0"/>
+    <axis xyz="0 0 1" />
+    <limit lower="-.002" upper="0" effort="100" velocity="100" />
+  </joint>
   <joint name="taskboard_lower/taskboard_slot1_switch3" type="revolute">
     <parent link="taskboard_slot1"/>
-    <child link="taskboard_slot1_switch3"/>
+    <child link="taskboard_slot1_switch3_pullout"/>
     <origin rpy=".47 0 0" xyz=".0005 -.089 0.009"/>
     <axis xyz="1 0 0"/>
     <limit effort="10000000.0" lower="-.94" upper="0" velocity="1000"/>
   </joint>
+  <joint name="taskboard_lower/taskboard_slot1_switch3_pullout" type="prismatic">
+    <parent link="taskboard_slot1_switch3_pullout"/>
+    <child link="taskboard_slot1_switch3"/>
+    <origin rpy="0 0 0" xyz="0 0 0"/>
+    <axis xyz="0 0 1" />
+    <limit lower="-.002" upper="0" effort="100" velocity="100" />
+  </joint>
   <joint name="taskboard_lower/taskboard_slot1_switch4" type="revolute">
     <parent link="taskboard_slot1"/>
-    <child link="taskboard_slot1_switch4"/>
+    <child link="taskboard_slot1_switch4_pullout"/>
     <origin rpy=".47 0 0" xyz=".0635 -.089 0.009"/>
     <axis xyz="1 0 0"/>
     <limit effort="10000000.0" lower="-.94" upper="0" velocity="1000"/>
+  </joint>
+  <joint name="taskboard_lower/taskboard_slot1_switch4_pullout" type="prismatic">
+    <parent link="taskboard_slot1_switch4_pullout"/>
+    <child link="taskboard_slot1_switch4"/>
+    <origin rpy="0 0 0" xyz="0 0 0"/>
+    <axis xyz="0 0 1" />
+    <limit lower="-.002" upper="0" effort="100" velocity="100" />
   </joint>
   <joint name="taskboard_lower/taskboard_slot1_switch1_cover" type="revolute">

Commit message: Added taskboard controller from TopCoder competition

File: r2_gazebo/urdf/taskboard.lower.xacro (robot description, xacro)
@@ -1,4 +1,4 @@
 <?xml version="1.0"?>
-<robot>
+<robot xmlns:controller="http://playerstage.sourceforge.net/gazebo/xmlschema/#controller">
   <link name="world"/>
   <link name="dummy">
@@ -220,5 +220,5 @@
     </collision>
     <inertial>
-      <mass value="5"/>
+      <mass value="0.5"/>
       <inertia ixx="1" ixy="0.0" ixz="0.0" iyy="1" iyz="0.0" izz="1"/>
     </inertial>
@@ -244,5 +244,5 @@
     </collision>
     <inertial>
-      <mass value="5"/>
+      <mass value="0.5"/>
       <inertia ixx="1" ixy="0.0" ixz="0.0" iyy="1" iyz="0.0" izz="1"/>
     </inertial>
@@ -268,5 +268,5 @@
     </collision>
     <inertial>
-      <mass value="5"/>
+      <mass value="0.5"/>
       <inertia ixx="1" ixy="0.0" ixz="0.0" iyy="1" iyz="0.0" izz="1"/>
     </inertial>
@@ -292,5 +292,5 @@
     </collision>
     <inertial>
-      <mass value="5"/>
+      <mass value="0.5"/>
       <inertia ixx="1" ixy="0.0" ixz="0.0" iyy="1" iyz="0.0" izz="1"/>
     </inertial>
@@ -310,5 +310,5 @@
     </collision>
     <inertial>
-      <mass value="5"/>
+      <mass value="0.5"/>
       <inertia ixx="1" ixy="0.0" ixz="0.0" iyy="1" iyz="0.0" izz="1"/>
     </inertial>
@@ -346,5 +346,5 @@
     </collision>
     <inertial>
-      <mass value="5"/>
+      <mass value="0.5"/>
       <inertia ixx="1" ixy="0.0" ixz="0.0" iyy="1" iyz="0.0" izz="1"/>
     </inertial>
@@ -364,5 +364,5 @@
     </collision>
     <inertial>
-      <mass value="5"/>
+      <mass value="0.5"/>
       <inertia ixx="1" ixy="0.0" ixz="0.0" iyy="1" iyz="0.0" izz="1"/>
     </inertial>
@@ -382,5 +382,5 @@
     </collision>
     <inertial>
-      <mass value="5"/>
+      <mass value="0.5"/>
       <inertia ixx="1" ixy="0.0" ixz="0.0" iyy="1" iyz="0.0" izz="1"/>
     </inertial>
@@ -400,5 +400,5 @@
     </collision>
     <inertial>
-      <mass value="5"/>
+      <mass value="0.5"/>
       <inertia ixx="1" ixy="0.0" ixz="0.0" iyy="1" iyz="0.0" izz="1"/>
     </inertial>
@@ -418,5 +418,5 @@
     </collision>
     <inertial>
-      <mass value="5"/>
+      <mass value="0.5"/>
       <inertia ixx="1" ixy="0.0" ixz="0.0" iyy="1" iyz="0.0" izz="1"/>
     </inertial>
@@ -436,5 +436,5 @@
     </collision>
     <inertial>
-      <mass value="5"/>
+      <mass value="0.5"/>
       <inertia ixx="1" ixy="0.0" ixz="0.0" iyy="1" iyz="0.0" izz="1"/>
     </inertial>
@@ -454,5 +454,5 @@
     </collision>
     <inertial>
-      <mass value="5"/>
+      <mass value="0.5"/>
       <inertia ixx="1" ixy="0.0" ixz="0.0" iyy="1" iyz="0.0" izz="1"/>
     </inertial>
@@ -472,5 +472,5 @@
     </collision>
     <inertial>
-      <mass value="5"/>
+      <mass value="0.5"/>
       <inertia ixx="1" ixy="0.0" ixz="0.0" iyy="1" iyz="0.0" izz="1"/>
     </inertial>
@@ -490,5 +490,5 @@
     </collision>
     <inertial>
-      <mass value="5"/>
+      <mass value="0.5"/>
       <inertia ixx="1" ixy="0.0" ixz="0.0" iyy="1" iyz="0.0" izz="1"/>
     </inertial>
@@ -526,5 +526,5 @@
     </collision>
     <inertial>
-      <mass value="5"/>
+      <mass value="0.5"/>
       <inertia ixx="1" ixy="0.0" ixz="0.0" iyy="1" iyz="0.0" izz="1"/>
     </inertial>
@@ -893,7 +893,7 @@
     <parent link="taskboard_slot1"/>
     <child link="taskboard_slot1_switch1"/>
-    <origin rpy="-.419 0 0" xyz=".037 .111 0.005"/>
+    <origin rpy="0.419 0 0" xyz=".037 .111 0.005"/>
     <axis xyz="1 0 0"/>
-    <limit effort="10000000.0" lower="0" upper=".84" velocity="1000"/>
+    <limit effort="10000000.0" lower="-0.84" upper="0" velocity="1000"/>
   </joint>
   <joint name="taskboard_lower/taskboard_slot1_switch2" type="revolute">
@@ -909,5 +909,5 @@
     <origin rpy="0 0 0" xyz="0 0 0"/>
     <axis xyz="0 0 1" />
-    <limit lower="-.002" upper="0" effort="100" velocity="100" />
+    <limit lower="-.002" upper="0.00" effort="100" velocity="100" />
   </joint>
   <joint name="taskboard_lower/taskboard_slot1_switch3" type="revolute">
@@ -955,5 +955,6 @@
     <child link="taskboard_slot1_A1"/>
     <origin rpy="0 0 0" xyz="0 0 0"/>
-    <limit lower="-.002" upper="0" effort="100" velocity="100" />
+    <axis xyz="0 0 1" />
+    <limit lower="-0.0005" upper="0.001" effort="100" velocity="100" />
   </joint>
   <joint name="taskboard_lower/taskboard_slot1_A2" type="prismatic">
@@ -961,5 +962,6 @@
     <child link="taskboard_slot1_A2"/>
     <origin rpy="0 0 0" xyz="0 0 0"/>
-    <limit lower="-.002" upper="0" effort="100" velocity="100" />
+    <axis xyz="0 0 1" />
+    <limit lower="-.0005" upper="0.001" effort="100" velocity="100" />
   </joint>
   <joint name="taskboard_lower/taskboard_slot1_A3" type="prismatic">
@@ -967,5 +969,6 @@
     <child link="taskboard_slot1_A3"/>
     <origin rpy="0 0 0" xyz="0 0 0"/>
-    <limit lower="-.002" upper="0" effort="100" velocity="100" />
+    <axis xyz="0 0 1" />
+    <limit lower="-.0005" upper="0.001" effort="100" velocity="100" />
   </joint>
   <joint name="taskboard_lower/taskboard_slot1_B1" type="prismatic">
@@ -973,5 +976,6 @@
     <child link="taskboard_slot1_B1"/>
     <origin rpy="0 0 0" xyz="0 0 0"/>
-    <limit lower="-.002" upper="0" effort="100" velocity="100" />
+    <axis xyz="0 0 1" />
+    <limit lower="-.0005" upper="0.001" effort="100" velocity="100" />
   </joint>
   <joint name="taskboard_lower/taskboard_slot1_B2" type="prismatic">
@@ -979,5 +983,6 @@
     <child link="taskboard_slot1_B2"/>
     <origin rpy="0 0 0" xyz="0 0 0"/>
-    <limit lower="-.002" upper="0" effort="100" velocity="100" />
+    <axis xyz="0 0 1" />
+    <limit lower="-.0005" upper="0.001" effort="100" velocity="100" />
   </joint>
   <joint name="taskboard_lower/taskboard_slot1_B3" type="prismatic">
@@ -985,5 +990,6 @@
     <child link="taskboard_slot1_B3"/>
     <origin rpy="0 0 0" xyz="0 0 0"/>
-    <limit lower="-.002" upper="0" effort="100" velocity="100" />
+    <axis xyz="0 0 1" />
+    <limit lower="-.0005" upper="0.001" effort="100" velocity="100" />
   </joint>
   <joint name="taskboard_lower/taskboard_slot1_C1" type="prismatic">
@@ -991,5 +997,6 @@
     <child link="taskboard_slot1_C1"/>
     <origin rpy="0 0 0" xyz="0 0 0"/>
-    <limit lower="-.002" upper="0" effort="100" velocity="100" />
+    <axis xyz="0 0 1" />
+    <limit lower="-.0005" upper="0.001" effort="100" velocity="100" />
   </joint>
   <joint name="taskboard_lower/taskboard_slot1_C2" type="prismatic">
@@ -997,5 +1004,6 @@
     <child link="taskboard_slot1_C2"/>
     <origin rpy="0 0 0" xyz="0 0 0"/>
-    <limit lower="-.002" upper="0" effort="100" velocity="100" />
+    <axis xyz="0 0 1" />
+    <limit lower="-.0005" upper="0.001" effort="100" velocity="100" />
   </joint>
   <joint name="taskboard_lower/taskboard_slot1_C3" type="prismatic">
@@ -1003,5 +1011,6 @@
     <child link="taskboard_slot1_C3"/>
     <origin rpy="0 0 0" xyz="0 0 0"/>
-    <limit lower="-.002" upper="0" effort="100" velocity="100" />
+    <axis xyz="0 0 1" />
+    <limit lower="-.0005" upper="0.001" effort="100" velocity="100" />
   </joint>
   <joint name="taskboard_lower/taskboard_slot1_blackplate" type="fixed">
@@ -1208,3 +1217,7 @@
     <material value="Gazebo/White" />
   </gazebo>
+  <gazebo>
+    <controller:gazebo_taskboard name="gazebo_taskboard" plugin="libgazebo_taskboard.so">
+    </controller:gazebo_taskboard>
+  </gazebo>
 </robot>
