Commit message: Subdivide taskboard urdf

File: r2_gazebo/urdf/taskboard.lower.xacro (robot description, xacro)
@@ -4,830 +4,10 @@
   <link name="dummy">
     <inertial>
-      <mass value="1"/>
+      <mass value="1" />
       <inertia ixx="1" ixy="0.0" ixz="0.0" iyy="1" iyz="0.0" izz="1"/>
     </inertial>
   </link>
-  <link name="taskboard_lower">
-    <visual>
-      <geometry>
-        <mesh filename="package://r2_gazebo/Media/models/taskboard/tskbd_lower_assembly_robonaut.dae"/>
-      </geometry>
-      <origin xyz="0.0 0.0 0.0" rpy="0 0 0"/>
-    </visual>
-    <collision>
-      <geometry>
-        <mesh filename="package://r2_gazebo/Media/models/taskboard/tskbd_lower_assembly_robonaut.dae" scale="0 0 0"/>
-      </geometry>
-      <origin xyz="0.0 0.0 0.0" rpy="0 0 0"/>
-    </collision>
-    <inertial>
-      <mass value="5"/>
-      <inertia ixx="1" ixy="0.0" ixz="0.0" iyy="1" iyz="0.0" izz="1"/>
-    </inertial>
-  </link>
-  <link name="taskboard_lower_labels">
-    <visual>
-      <geometry>
-        <mesh filename="package://r2_gazebo/Media/models/taskboard/tskbd_lower_assembly_labels.dae"/>
-      </geometry>
-      <origin xyz="0.0 0.0 0.0" rpy="0 0 0"/>
-    </visual>
-    <collision>
-      <geometry>
-        <mesh filename="package://r2_gazebo/Media/models/taskboard/tskbd_lower_assembly_labels.dae" scale="0 0 0"/>
-      </geometry>
-      <origin xyz="0.0 0.0 0.0" rpy="0 0 0"/>
-    </collision>
-    <inertial>
-      <mass value="5"/>
-      <inertia ixx="1" ixy="0.0" ixz="0.0" iyy="1" iyz="0.0" izz="1"/>
-    </inertial>
-  </link>
-  <link name="taskboard_slot3">
-    <visual>
-      <geometry>
-        <mesh filename="package://r2_gazebo/Media/models/taskboard/tskbd_panel_assembly_eva_slot3.dae"/>
-      </geometry>
-      <origin xyz="0.0 0.0 0.0" rpy="0 0 0"/>
-    </visual>
-    <collision>
-      <geometry>
-        <mesh filename="package://r2_gazebo/Media/models/taskboard/tskbd_panel_assembly_eva_slot3.dae" scale="1 1 1"/>
-      </geometry>
-      <origin xyz="0.0 0.0 0.0" rpy="0 0 0"/>
-    </collision>
-    <inertial>
-      <mass value="5"/>
-      <inertia ixx="1" ixy="0.0" ixz="0.0" iyy="1" iyz="0.0" izz="1"/>
-    </inertial>
-  </link>
-  <link name="taskboard_slot3_panel">
-    <visual>
-      <geometry>
-        <mesh filename="package://r2_gazebo/Media/models/taskboard/tskbd_panel_assembly_slot1_panel.dae"/>
-      </geometry>
-      <origin xyz="0.0 0.0 0.0" rpy="0 0 0"/>
-    </visual>
-    <collision>
-      <geometry>
-        <mesh filename="package://r2_gazebo/Media/models/taskboard/tskbd_panel_assembly_slot1_panel.dae" scale="1 1 1"/>
-      </geometry>
-      <origin xyz="0.0 0.0 0.0" rpy="0 0 0"/>
-    </collision>
-    <inertial>
-      <mass value="5"/>
-      <inertia ixx="1" ixy="0.0" ixz="0.0" iyy="1" iyz="0.0" izz="1"/>
-    </inertial>
-  </link>
-  <link name="taskboard_slot3_labels">
-    <visual>
-      <geometry>
-        <mesh filename="package://r2_gazebo/Media/models/taskboard/tskbd_panel_assembly_eva_slot3_labels.dae"/>
-      </geometry>
-      <origin xyz="0.0 0.0 0.0" rpy="0 0 0"/>
-    </visual>
-    <collision>
-      <geometry>
-        <mesh filename="package://r2_gazebo/Media/models/taskboard/tskbd_panel_assembly_eva_slot3_labels.dae" scale="1 1 1"/>
-      </geometry>
-      <origin xyz="0.0 0.0 0.0" rpy="0 0 0"/>
-    </collision>
-    <inertial>
-      <mass value="5"/>
-      <inertia ixx="1" ixy="0.0" ixz="0.0" iyy="1" iyz="0.0" izz="1"/>
-    </inertial>
-  </link>
-  <link name="taskboard_slot4">
-    <visual>
-      <geometry>
-        <mesh filename="package://r2_gazebo/Media/models/taskboard/tskbd_panel_assembly_slot4.dae"/>
-      </geometry>
-      <origin xyz="0.0 0.0 0.0" rpy="0 0 0"/>
-    </visual>
-    <collision>
-      <geometry>
-        <mesh filename="package://r2_gazebo/Media/models/taskboard/tskbd_panel_assembly_slot4.dae" scale="1 1 1"/>
-      </geometry>
-      <origin xyz="0.0 0.0 0.0" rpy="0 0 0"/>
-    </collision>
-    <inertial>
-      <mass value="5"/>
-      <inertia ixx="1" ixy="0.0" ixz="0.0" iyy="1" iyz="0.0" izz="1"/>
-    </inertial>
-  </link>
-  <link name="taskboard_slot4_panel">
-    <visual>
-      <geometry>
-        <mesh filename="package://r2_gazebo/Media/models/taskboard/tskbd_panel_assembly_slot4_panel.dae"/>
-      </geometry>
-      <origin xyz="0.0 0.0 0.0" rpy="0 0 0"/>
-    </visual>
-    <collision>
-      <geometry>
-        <mesh filename="package://r2_gazebo/Media/models/taskboard/tskbd_panel_assembly_slot4_panel.dae" scale="1 1 1"/>
-      </geometry>
-      <origin xyz="0.0 0.0 0.0" rpy="0 0 0"/>
-    </collision>
-    <inertial>
-      <mass value="5"/>
-      <inertia ixx="1" ixy="0.0" ixz="0.0" iyy="1" iyz="0.0" izz="1"/>
-    </inertial>
-  </link>
-  <link name="taskboard_slot4_labels">
-    <visual>
-      <geometry>
-        <mesh filename="package://r2_gazebo/Media/models/taskboard/tskbd_panel_assembly_slot4_labels.dae"/>
-      </geometry>
-      <origin xyz="0.0 0.0 0.0" rpy="0 0 0"/>
-    </visual>
-    <collision>
-      <geometry>
-        <mesh filename="package://r2_gazebo/Media/models/taskboard/tskbd_panel_assembly_slot4_labels.dae" scale="1 1 1"/>
-      </geometry>
-      <origin xyz="0.0 0.0 0.0" rpy="0 0 0"/>
-    </collision>
-    <inertial>
-      <mass value="5"/>
-      <inertia ixx="1" ixy="0.0" ixz="0.0" iyy="1" iyz="0.0" izz="1"/>
-    </inertial>
-  </link>
-  <link name="taskboard_slot1">
-    <visual>
-      <geometry>
-        <mesh filename="package://r2_gazebo/Media/models/taskboard/tskbd_panel_assembly_slot1.dae"/>
-      </geometry>
-      <origin xyz="0.0 0.0 0.0" rpy="0 0 0"/>
-    </visual>
-    <collision>
-      <geometry>
-        <mesh filename="package://r2_gazebo/Media/models/taskboard/tskbd_panel_assembly_slot1.dae" scale="1 1 1"/>
-      </geometry>
-      <origin xyz="0.0 0.0 0.0" rpy="0 0 0"/>
-    </collision>
-    <inertial>
-      <mass value="5"/>
-      <inertia ixx="1" ixy="0.0" ixz="0.0" iyy="1" iyz="0.0" izz="1"/>
-    </inertial>
-  </link>
-  <link name="taskboard_slot1_panel">
-    <visual>
-      <geometry>
-        <mesh filename="package://r2_gazebo/Media/models/taskboard/tskbd_panel_assembly_slot1_panel.dae"/>
-      </geometry>
-      <origin xyz="0.0 0.0 0.0" rpy="0 0 0"/>
-    </visual>
-    <collision>
-      <geometry>
-        <mesh filename="package://r2_gazebo/Media/models/taskboard/tskbd_panel_assembly_slot1_panel.dae" scale="1 1 1"/>
-      </geometry>
-      <origin xyz="0.0 0.0 0.0" rpy="0 0 0"/>
-    </collision>
-    <inertial>
-      <mass value="5"/>
-      <inertia ixx="1" ixy="0.0" ixz="0.0" iyy="1" iyz="0.0" izz="1"/>
-    </inertial>
-  </link>
-  <link name="taskboard_slot1_labels">
-    <visual>
-      <geometry>
-        <mesh filename="package://r2_gazebo/Media/models/taskboard/tskbd_panel_assembly_slot1_labels.dae"/>
-      </geometry>
-      <origin xyz="0.0 0.0 0.0" rpy="0 0 0"/>
-    </visual>
-    <collision>
-      <geometry>
-        <mesh filename="package://r2_gazebo/Media/models/taskboard/tskbd_panel_assembly_slot1_labels.dae" scale="1 1 1"/>
-      </geometry>
-      <origin xyz="0.0 0.0 0.0" rpy="0 0 0"/>
-    </collision>
-    <inertial>
-      <mass value="5"/>
-      <inertia ixx="1" ixy="0.0" ixz="0.0" iyy="1" iyz="0.0" izz="1"/>
-    </inertial>
-  </link>
-  <link name="taskboard_slot1_switch1">
-    <visual>
-      <geometry>
-        <mesh filename="package://r2_gazebo/Media/models/taskboard/tskbd_panel_assembly_slot1_switch1.dae"/>
-      </geometry>
-      <origin xyz="0.0 0.0 0.0" rpy="0 0 0"/>
-    </visual>
-    <collision>
-      <geometry>
-        <mesh filename="package://r2_gazebo/Media/models/taskboard/tskbd_panel_assembly_slot1_switch1.dae" scale="1 1 1"/>
-      </geometry>
-      <origin xyz="0.0 0.0 0.0" rpy="0 0 0"/>
-    </collision>
-    <inertial>
-      <mass value="0.5"/>
-      <inertia ixx="1" ixy="0.0" ixz="0.0" iyy="1" iyz="0.0" izz="1"/>
-    </inertial>
-  </link>
-  <link name="taskboard_slot1_switch2_pullout">
-    <inertial>
-      <mass value=".01"/>
-      <inertia ixx="1" ixy="0.0" ixz="0.0" iyy="1" iyz="0.0" izz="1"/>
-    </inertial>
-  </link>
-  <link name="taskboard_slot1_switch2">
-    <visual>
-      <geometry>
-        <mesh filename="package://r2_gazebo/Media/models/taskboard/tskbd_panel_assembly_slot1_switch2.dae"/>
-      </geometry>
-      <origin xyz="0.0 0.0 0.0" rpy="0 0 0"/>
-    </visual>
-    <collision>
-      <geometry>
-        <mesh filename="package://r2_gazebo/Media/models/taskboard/tskbd_panel_assembly_slot1_switch2.dae" scale="1 1 1"/>
-      </geometry>
-      <origin xyz="0.0 0.0 0.0" rpy="0 0 0"/>
-    </collision>
-    <inertial>
-      <mass value="0.5"/>
-      <inertia ixx="1" ixy="0.0" ixz="0.0" iyy="1" iyz="0.0" izz="1"/>
-    </inertial>
-  </link>
-  <link name="taskboard_slot1_switch3_pullout">
-    <inertial>
-      <mass value=".01"/>
-      <inertia ixx="1" ixy="0.0" ixz="0.0" iyy="1" iyz="0.0" izz="1"/>
-    </inertial>
-  </link>
-  <link name="taskboard_slot1_switch3">
-    <visual>
-      <geometry>
-        <mesh filename="package://r2_gazebo/Media/models/taskboard/tskbd_panel_assembly_slot1_switch3.dae"/>
-      </geometry>
-      <origin xyz="0.0 0.0 0.0" rpy="0 0 0"/>
-    </visual>
-    <collision>
-      <geometry>
-        <mesh filename="package://r2_gazebo/Media/models/taskboard/tskbd_panel_assembly_slot1_switch3.dae" scale="1 1 1"/>
-      </geometry>
-      <origin xyz="0.0 0.0 0.0" rpy="0 0 0"/>
-    </collision>
-    <inertial>
-      <mass value="0.5"/>
-      <inertia ixx="1" ixy="0.0" ixz="0.0" iyy="1" iyz="0.0" izz="1"/>
-    </inertial>
-  </link>
-  <link name="taskboard_slot1_switch4_pullout">
-    <inertial>
-      <mass value=".01"/>
-      <inertia ixx="1" ixy="0.0" ixz="0.0" iyy="1" iyz="0.0" izz="1"/>
-    </inertial>
-  </link>
-  <link name="taskboard_slot1_switch4">
-    <visual>
-      <geometry>
-        <mesh filename="package://r2_gazebo/Media/models/taskboard/tskbd_panel_assembly_slot1_switch4.dae"/>
-      </geometry>
-      <origin xyz="0.0 0.0 0.0" rpy="0 0 0"/>
-    </visual>
-    <collision>
-      <geometry>
-        <mesh filename="package://r2_gazebo/Media/models/taskboard/tskbd_panel_assembly_slot1_switch4.dae" scale="1 1 1"/>
-      </geometry>
-      <origin xyz="0.0 0.0 0.0" rpy="0 0 0"/>
-    </collision>
-    <inertial>
-      <mass value="0.5"/>
-      <inertia ixx="1" ixy="0.0" ixz="0.0" iyy="1" iyz="0.0" izz="1"/>
-    </inertial>
-  </link>
-  <link name="taskboard_slot1_switch1_cover">
-    <visual>
-      <geometry>
-        <mesh filename="package://r2_gazebo/Media/models/taskboard/tskbd_panel_assembly_slot1_switch1_cover.dae"/>
-      </geometry>
-      <origin xyz="0.0 0.0 0.0" rpy="0 0 0"/>
-    </visual>
-    <collision>
-      <geometry>
-        <mesh filename="package://r2_gazebo/Media/models/taskboard/tskbd_panel_assembly_slot1_switch1_cover.dae" scale="1 1 1"/>
-      </geometry>
-      <origin xyz="0.0 0.0 0.0" rpy="0 0 0"/>
-    </collision>
-    <inertial>
-      <mass value="0.5"/>
-      <inertia ixx="1" ixy="0.0" ixz="0.0" iyy="1" iyz="0.0" izz="1"/>
-    </inertial>
-  </link>
-  <link name="taskboard_slot1_guard">
-    <visual>
-      <geometry>
-        <mesh filename="package://r2_gazebo/Media/models/taskboard/tskbd_panel_assembly_slot1_guard.dae"/>
-      </geometry>
-      <origin xyz="0.0 0.0 0.0" rpy="0 0 0"/>
-    </visual>
-    <collision>
-      <geometry>
-        <mesh filename="package://r2_gazebo/Media/models/taskboard/tskbd_panel_assembly_slot1_guard.dae" scale="1 1 1"/>
-      </geometry>
-      <origin xyz="0.0 0.0 0.0" rpy="0 0 0"/>
-    </collision>
-    <inertial>
-      <mass value="5"/>
-      <inertia ixx="1" ixy="0.0" ixz="0.0" iyy="1" iyz="0.0" izz="1"/>
-    </inertial>
-  </link>
-  <link name="taskboard_slot1_A1">
-    <visual>
-      <geometry>
-        <mesh filename="package://r2_gazebo/Media/models/taskboard/tskbd_panel_assembly_slot1_a1.dae"/>
-      </geometry>
-      <origin xyz="0.0 0.0 0.0" rpy="0 0 0"/>
-    </visual>
-    <collision>
-      <geometry>
-        <mesh filename="package://r2_gazebo/Media/models/taskboard/tskbd_panel_assembly_slot1_a1.dae" scale="1 1 1"/>
-      </geometry>
-      <origin xyz="0.0 0.0 0.0" rpy="0 0 0"/>
-    </collision>
-    <inertial>
-      <mass value="0.5"/>
-      <inertia ixx="1" ixy="0.0" ixz="0.0" iyy="1" iyz="0.0" izz="1"/>
-    </inertial>
-  </link>
-  <link name="taskboard_slot1_A2">
-    <visual>
-      <geometry>
-        <mesh filename="package://r2_gazebo/Media/models/taskboard/tskbd_panel_assembly_slot1_a2.dae"/>
-      </geometry>
-      <origin xyz="0.0 0.0 0.0" rpy="0 0 0"/>
-    </visual>
-    <collision>
-      <geometry>
-        <mesh filename="package://r2_gazebo/Media/models/taskboard/tskbd_panel_assembly_slot1_a2.dae" scale="1 1 1"/>
-      </geometry>
-      <origin xyz="0.0 0.0 0.0" rpy="0 0 0"/>
-    </collision>
-    <inertial>
-      <mass value="0.5"/>
-      <inertia ixx="1" ixy="0.0" ixz="0.0" iyy="1" iyz="0.0" izz="1"/>
-    </inertial>
-  </link>
-  <link name="taskboard_slot1_A3">
-    <visual>
-      <geometry>
-        <mesh filename="package://r2_gazebo/Media/models/taskboard/tskbd_panel_assembly_slot1_a3.dae"/>
-      </geometry>
-      <origin xyz="0.0 0.0 0.0" rpy="0 0 0"/>
-    </visual>
-    <collision>
-      <geometry>
-        <mesh filename="package://r2_gazebo/Media/models/taskboard/tskbd_panel_assembly_slot1_a3.dae" scale="1 1 1"/>
-      </geometry>
-      <origin xyz="0.0 0.0 0.0" rpy="0 0 0"/>
-    </collision>
-    <inertial>
-      <mass value="0.5"/>
-      <inertia ixx="1" ixy="0.0" ixz="0.0" iyy="1" iyz="0.0" izz="1"/>
-    </inertial>
-  </link>
-  <link name="taskboard_slot1_B1">
-    <visual>
-      <geometry>
-        <mesh filename="package://r2_gazebo/Media/models/taskboard/tskbd_panel_assembly_slot1_b1.dae"/>
-      </geometry>
-      <origin xyz="0.0 0.0 0.0" rpy="0 0 0"/>
-    </visual>
-    <collision>
-      <geometry>
-        <mesh filename="package://r2_gazebo/Media/models/taskboard/tskbd_panel_assembly_slot1_b1.dae" scale="1 1 1"/>
-      </geometry>
-      <origin xyz="0.0 0.0 0.0" rpy="0 0 0"/>
-    </collision>
-    <inertial>
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
File: r2_gazebo/urdf/taskboard.urdf.xacro (robot description, xacro)
@@ -1,7 +1,43 @@
 <?xml version="1.0" ?>
 <robot name="taskboard" xmlns:xacro="http://wiki.ros.org/xacro">
+    <xacro:macro name="std_mesh" params="name mesh mass">
+      <link name="${name}">
+        <visual>
+          <geometry>
+            <mesh filename="package://r2_gazebo/Media/models/taskboard/${mesh}"/>
+          </geometry> <material name="black">
+        <color rgba="0 0 0 1"/>
+      </material>
+        </visual>
+        <collision>
+          <geometry>
+            <mesh filename="package://r2_gazebo/Media/models/taskboard/${mesh}"/>
+          </geometry>
+        </collision>
+        <inertial>
+          <mass value="${mass}"/>
+          <inertia ixx="1" ixy="0.0" ixz="0.0" iyy="1" iyz="0.0" izz="1"/>
+        </inertial>
+      </link>
+    </xacro:macro>
+    <xacro:macro name="mesh_no_collide" params="name mesh mass">
+      <link name="${name}">
+        <visual>
+          <geometry>
+            <mesh filename="package://r2_gazebo/Media/models/taskboard/${mesh}"/>
+          </geometry>
+        </visual>
+        <collision>
+          <geometry>
+            <mesh filename="package://r2_gazebo/Media/models/taskboard/${mesh}" scale="0 0 0"/>
+          </geometry>
+        </collision>
+        <inertial>
+          <mass value="${mass}"/>
+          <inertia ixx="1" ixy="0.0" ixz="0.0" iyy="1" iyz="0.0" izz="1"/>
+        </inertial>
+      </link>
+    </xacro:macro>
   <xacro:include filename="$(find r2_gazebo)/urdf/taskboard.lower.xacro" />
-  <xacro:include filename="$(find r2_gazebo)/urdf/taskboard.B01.xacro" />
-  <xacro:include filename="$(find r2_gazebo)/urdf/taskboard.B05.xacro" />
   <xacro:include filename="$(find r2_gazebo)/urdf/gazebo_plugins/gazebo_interface.xacro" />
   <xacro:include filename="$(find r2_gazebo)/urdf/gazebo_plugins/taskboard.panel_a.controller.xacro" />
